File: MicroSDv2/MicroSDv2.sch (KiCad schematic (older format))
At the start: 14 parts, among them J1 Conn_01x08, J3 Micro_SD_Card_Det, U1 AP7365, U2 4050

Commit message: Part Numbers Added
Parts:
- C1, C2: Part (none) -> C29936
- D1: Part (none) -> C118330
- J3: Part (none) -> C114218
- R1: Part (none) -> C227816
- R3: Part (none) -> C99198
- R6: Part (none) -> C25585
- U2: Part (none) -> C352821
Other:
- moved on the sheet: C1, C2, D1, H1, H2, H3, H4, J1, J3, R1, R3, R6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
