File: QFN20/QFN20.sch (KiCad schematic (older format))
At the start: 4 parts, among them J1 Conn_01x10, J2 Conn_02x10_Counter_Clockwise, J3 Conn_01x10, J4 Conn_02x10_Counter_Clockwise

Commit message: Silkscreens and sizes updated
Parts:
- added J5: Conn_01x03, Connector_PinHeader_2.54mm:PinHeader_1x03_P2.54mm_Vertical, symbol Connector_Generic:Conn_01x03
Connections:
- new net: J5.1 (Pin_1), J5.2 (Pin_2), J5.3 (Pin_3)
Changed lines of the file:
@@
 Connection ~ 5600 4700
 Connection ~ 5600 4800
+$Comp
+L Connector_Generic:Conn_01x03 J5
+U 1 1 5D3B65EC
+P 7600 4300
+F 0 "J5" H 7679 4342 50  0000 L CNN
+F 1 "Conn_01x03" H 7679 4252 50  0000 L CNN
+F 2 "Connector_PinHeader_2.54mm:PinHeader_1x03_P2.54mm_Vertical" H 7600 4300 50  0001 C CNN
+F 3 "~" H 7600 4300 50  0001 C CNN
+	1    7600 4300
+	1    0    0    -1
+$EndComp
+Wire Wire Line
+	7400 4200 7400 4300
+Connection ~ 7400 4300
+Wire Wire Line
+	7400 4300 7400 4400
 $EndSCHEMATC

Commit message: Page Settings Updated
Other:
- moved on the sheet: J1, J2, J3, J4, J5
Changed lines of the file:
@@
 EELAYER 29 0
 EELAYER END
-$Descr A4 11693 8268
+$Descr User 8268 5807
 encoding utf-8
 Sheet 1 1
@@
 L Connector_Generic:Conn_01x10 J3
 U 1 1 5D27A585
-P 5800 4300
-F 0 "J3" H 5879 4292 50  0000 L CNN
-F 1 "Conn_01x10" H 5879 4202 50  0000 L CNN
-F 2 "Connector_PinHeader_2.54mm:PinHeader_1x10_P2.54mm_Vertical" H 5800 4300 50  0001 C CNN
-F 3 "~" H 5800 4300 50  0001 C CNN
-	1    5800 4300
+P 3750 2500
+F 0 "J3" H 3829 2492 50  0000 L CNN
+F 1 "Conn_01x10" H 3829 2402 50  0000 L CNN
+F 2 "Connector_PinHeader_2.54mm:PinHeader_1x10_P2.54mm_Vertical" H 3750 2500 50  0001 C CNN
+F 3 "~" H 3750 2500 50  0001 C CNN
+	1    3750 2500
 	1    0    0    -1
 $EndComp
@@
 L Connector_Generic:Conn_02x10_Counter_Clockwise J2
 U 1 1 5D27AA24
-P 5300 4300
-F 0 "J2" H 5350 4915 50  0000 C CNN
-F 1 "Conn_02x10_Counter_Clockwise" H 5350 4825 50  0000 C CNN
-F 2 "Package_DFN_QFN:QFN-20-1EP_4x4mm_P0.5mm_EP2.5x2.5mm" H 5300 4300 50  0001 C CNN
-F 3 "~" H 5300 4300 50  0001 C CNN
-	1    5300 4300
+P 3250 2500
+F 0 "J2" H 3300 3115 50  0000 C CNN
+F 1 "Conn_02x10_Counter_Clockwise" H 3300 3025 50  0000 C CNN
+F 2 "Package_DFN_QFN:QFN-20-1EP_4x4mm_P0.5mm_EP2.5x2.5mm" H 3250 2500 50  0001 C CNN
+F 3 "~" H 3250 2500 50  0001 C CNN
+	1    3250 2500
 	1    0    0    -1
 $EndComp
@@
 L Connector_Generic:Conn_01x10 J1
 U 1 1 5D27D08B
-P 4900 4300
-F 0 "J1" H 4979 4292 50  0000 L CNN
-F 1 "Conn_01x10" H 4979 4202 50  0000 L CNN
-F 2 "Connector_PinHeader_2.54mm:PinHeader_1x10_P2.54mm_Vertical" H 4900 4300 50  0001 C CNN
-F 3 "~" H 4900 4300 50  0001 C CNN
-	1    4900 4300
+P 2850 2500
+F 0 "J1" H 2929 2492 50  0000 L CNN
+F 1 "Conn_01x10" H 2929 2402 50  0000 L CNN
+F 2 "Connector_PinHeader_2.54mm:PinHeader_1x10_P2.54mm_Vertical" H 2850 2500 50  0001 C CNN
+F 3 "~" H 2850 2500 50  0001 C CNN
+	1    2850 2500
 	-1   0    0    -1
 $EndComp
@@
 L Connector_Generic:Conn_02x10_Counter_Clockwise J4
 U 1 1 5D287A35
-P 5300 4400
-F 0 "J4" H 5350 5015 50  0000 C CNN
-F 1 "Conn_02x10_Counter_Clockwise" H 5350 4925 50  0000 C CNN
-F 2 "Package_DFN_QFN:QFN-20-1EP_5x5mm_P0.65mm_EP3.35x3.35mm" H 5300 4400 50  0001 C CNN
-F 3 "~" H 5300 4400 50  0001 C CNN
-	1    5300 4400
+P 3250 2600
+F 0 "J4" H 3300 3215 50  0000 C CNN
+F 1 "Conn_02x10_Counter_Clockwise" H 3300 3125 50  0000 C CNN
+F 2 "Package_DFN_QFN:QFN-20-1EP_5x5mm_P0.65mm_EP3.35x3.35mm" H 3250 2600 50  0001 C CNN
+F 3 "~" H 3250 2600 50  0001 C CNN
+	1    3250 2600
 	1    0    0    1
 $EndComp
-Connection ~ 5100 3900
-Connection ~ 5100 4000
-Connection ~ 5100 4100
-Connection ~ 5100 4200
-Connection ~ 5100 4300
-Connection ~ 5100 4400
-Connection ~ 5100 4500
-Connection ~ 5100 4600
-Connection ~ 5100 4700
-Connection ~ 5100 4800
-Connection ~ 5600 3900
-Connection ~ 5600 4000
-Connection ~ 5600 4100
-Connection ~ 5600 4200
-Connection ~ 5600 4300
-Connection ~ 5600 4400
-Connection ~ 5600 4500
-Connection ~ 5600 4600
-Connection ~ 5600 4700
-Connection ~ 5600 4800
+Connection ~ 3050 2100
+Connection ~ 3050 2200
+Connection ~ 3050 2300
+Connection ~ 3050 2400
+Connection ~ 3050 2500
+Connection ~ 3050 2600
+Connection ~ 3050 2700
+Connection ~ 3050 2800
+Connection ~ 3050 2900
+Connection ~ 3050 3000
+Connection ~ 3550 2100
+Connection ~ 3550 2200
+Connection ~ 3550 2300
+Connection ~ 3550 2400
+Connection ~ 3550 2500
+Connection ~ 3550 2600
+Connection ~ 3550 2700
+Connection ~ 3550 2800
+Connection ~ 3550 2900
+Connection ~ 3550 3000
 $Comp
 L Connector_Generic:Conn_01x03 J5
 U 1 1 5D3B65EC
-P 7600 4300
-F 0 "J5" H 7679 4342 50  0000 L CNN
-F 1 "Conn_01x03" H 7679 4252 50  0000 L CNN
-F 2 "Connector_PinHeader_2.54mm:PinHeader_1x03_P2.54mm_Vertical" H 7600 4300 50  0001 C CNN
-F 3 "~" H 7600 4300 50  0001 C CNN
-	1    7600 4300
+P 5550 2500
+F 0 "J5" H 5629 2542 50  0000 L CNN
+F 1 "Conn_01x03" H 5629 2452 50  0000 L CNN
+F 2 "Connector_PinHeader_2.54mm:PinHeader_1x03_P2.54mm_Vertical" H 5550 2500 50  0001 C CNN
+F 3 "~" H 5550 2500 50  0001 C CNN
+	1    5550 2500
 	1    0    0    -1
 $EndComp
 Wire Wire Line
-	7400 4200 7400 4300
-Connection ~ 7400 4300
+	5350 2400 5350 2500
+Connection ~ 5350 2500
 Wire Wire Line
-	7400 4300 7400 4400
+	5350 2500 5350 2600
 $EndSCHEMATC

Commit message: Schematic PDF and 3D Renders added
Other:
- moved on the sheet: J1, J2, J3, J4, J5
Changed lines of the file:
@@
 EELAYER 29 0
 EELAYER END
-$Descr User 8268 5807
+$Descr User 5197 4016
 encoding utf-8
 Sheet 1 1
@@
 L Connector_Generic:Conn_01x10 J3
 U 1 1 5D27A585
-P 3750 2500
-F 0 "J3" H 3829 2492 50  0000 L CNN
-F 1 "Conn_01x10" H 3829 2402 50  0000 L CNN
-F 2 "Connector_PinHeader_2.54mm:PinHeader_1x10_P2.54mm_Vertical" H 3750 2500 50  0001 C CNN
-F 3 "~" H 3750 2500 50  0001 C CNN
-	1    3750 2500
+P 2600 1375
+F 0 "J3" H 2679 1367 50  0000 L CNN
+F 1 "Conn_01x10" H 2679 1277 50  0000 L CNN
+F 2 "Connector_PinHeader_2.54mm:PinHeader_1x10_P2.54mm_Vertical" H 2600 1375 50  0001 C CNN
+F 3 "~" H 2600 1375 50  0001 C CNN
+	1    2600 1375
 	1    0    0    -1
 $EndComp
@@
 L Connector_Generic:Conn_02x10_Counter_Clockwise J2
 U 1 1 5D27AA24
-P 3250 2500
-F 0 "J2" H 3300 3115 50  0000 C CNN
-F 1 "Conn_02x10_Counter_Clockwise" H 3300 3025 50  0000 C CNN
-F 2 "Package_DFN_QFN:QFN-20-1EP_4x4mm_P0.5mm_EP2.5x2.5mm" H 3250 2500 50  0001 C CNN
-F 3 "~" H 3250 2500 50  0001 C CNN
-	1    3250 2500
+P 2100 1375
+F 0 "J2" H 2150 1990 50  0000 C CNN
+F 1 "Conn_02x10_Counter_Clockwise" H 2150 1900 50  0000 C CNN
+F 2 "Package_DFN_QFN:QFN-20-1EP_4x4mm_P0.5mm_EP2.5x2.5mm" H 2100 1375 50  0001 C CNN
+F 3 "~" H 2100 1375 50  0001 C CNN
+	1    2100 1375
 	1    0    0    -1
 $EndComp
@@
 L Connector_Generic:Conn_01x10 J1
 U 1 1 5D27D08B
-P 2850 2500
-F 0 "J1" H 2929 2492 50  0000 L CNN
-F 1 "Conn_01x10" H 2929 2402 50  0000 L CNN
-F 2 "Connector_PinHeader_2.54mm:PinHeader_1x10_P2.54mm_Vertical" H 2850 2500 50  0001 C CNN
-F 3 "~" H 2850 2500 50  0001 C CNN
-	1    2850 2500
+P 1700 1375
+F 0 "J1" H 1779 1367 50  0000 L CNN
+F 1 "Conn_01x10" H 1779 1277 50  0000 L CNN
+F 2 "Connector_PinHeader_2.54mm:PinHeader_1x10_P2.54mm_Vertical" H 1700 1375 50  0001 C CNN
+F 3 "~" H 1700 1375 50  0001 C CNN
+	1    1700 1375
 	-1   0    0    -1
 $EndComp
@@
 L Connector_Generic:Conn_02x10_Counter_Clockwise J4
 U 1 1 5D287A35
-P 3250 2600
-F 0 "J4" H 3300 3215 50  0000 C CNN
-F 1 "Conn_02x10_Counter_Clockwise" H 3300 3125 50  0000 C CNN
-F 2 "Package_DFN_QFN:QFN-20-1EP_5x5mm_P0.65mm_EP3.35x3.35mm" H 3250 2600 50  0001 C CNN
-F 3 "~" H 3250 2600 50  0001 C CNN
-	1    3250 2600
+P 2100 1475
+F 0 "J4" H 2150 2090 50  0000 C CNN
+F 1 "Conn_02x10_Counter_Clockwise" H 2150 2000 50  0000 C CNN
+F 2 "Package_DFN_QFN:QFN-20-1EP_5x5mm_P0.65mm_EP3.35x3.35mm" H 2100 1475 50  0001 C CNN
+F 3 "~" H 2100 1475 50  0001 C CNN
+	1    2100 1475
 	1    0    0    1
 $EndComp
-Connection ~ 3050 2100
-Connection ~ 3050 2200
-Connection ~ 3050 2300
-Connection ~ 3050 2400
-Connection ~ 3050 2500
-Connection ~ 3050 2600
-Connection ~ 3050 2700
-Connection ~ 3050 2800
-Connection ~ 3050 2900
-Connection ~ 3050 3000
-Connection ~ 3550 2100
-Connection ~ 3550 2200
-Connection ~ 3550 2300
-Connection ~ 3550 2400
-Connection ~ 3550 2500
-Connection ~ 3550 2600
-Connection ~ 3550 2700
-Connection ~ 3550 2800
-Connection ~ 3550 2900
-Connection ~ 3550 3000
+Connection ~ 1900 975
+Connection ~ 1900 1075
+Connection ~ 1900 1175
+Connection ~ 1900 1275
+Connection ~ 1900 1375
+Connection ~ 1900 1475
+Connection ~ 1900 1575
+Connection ~ 1900 1675
+Connection ~ 1900 1775
+Connection ~ 1900 1875
+Connection ~ 2400 975
+Connection ~ 2400 1075
+Connection ~ 2400 1175
+Connection ~ 2400 1275
+Connection ~ 2400 1375
+Connection ~ 2400 1475
+Connection ~ 2400 1575
+Connection ~ 2400 1675
+Connection ~ 2400 1775
+Connection ~ 2400 1875
 $Comp
 L Connector_Generic:Conn_01x03 J5
 U 1 1 5D3B65EC
-P 5550 2500
-F 0 "J5" H 5629 2542 50  0000 L CNN
-F 1 "Conn_01x03" H 5629 2452 50  0000 L CNN
-F 2 "Connector_PinHeader_2.54mm:PinHeader_1x03_P2.54mm_Vertical" H 5550 2500 50  0001 C CNN
-F 3 "~" H 5550 2500 50  0001 C CNN
-	1    5550 2500
+P 3900 1475
+F 0 "J5" H 3979 1517 50  0000 L CNN
+F 1 "Conn_01x03" H 3979 1427 50  0000 L CNN
+F 2 "Connector_PinHeader_2.54mm:PinHeader_1x03_P2.54mm_Vertical" H 3900 1475 50  0001 C CNN
+F 3 "~" H 3900 1475 50  0001 C CNN
+	1    3900 1475
 	1    0    0    -1
 $EndComp
 Wire Wire Line
-	5350 2400 5350 2500
-Connection ~ 5350 2500
+	3700 1375 3700 1475
+Connection ~ 3700 1475
 Wire Wire Line
-	5350 2500 5350 2600
+	3700 1475 3700 1575
 $EndSCHEMATC
