File: CR2032/CR2032.sch (KiCad schematic (older format))
At the start: 6 parts, among them J1 Conn_01x06

Commit message: Part Numbers Added
Parts:
- BT1: Part (none) -> C238100
Changed lines of the file:
@@
 F 2 "Battery:BatteryHolder_Keystone_3008_1x2450" V 2200 1510 50  0001 C CNN
 F 3 "~" V 2200 1510 50  0001 C CNN
+F 4 "C238100" H 2200 1450 50  0001 C CNN "Part"
 	1    2200 1450
 	1    0    0    -1

Commit message: Board size updated
Board size changed from 33.02mmX26.035mm to 33.02mmX25.4mm
Parts:
- H1, H2, H3, H4: footprint MountingHole:MountingHole_2.7mm_M2.5_ISO14580_Pad -> SirBoardLibrary:MountingHole_M2.5_SirBoard
Changed lines of the file:
@@
 F 0 "H1" H 3150 845 50  0000 L CNN
 F 1 "MountingHole" H 3150 755 50  0000 L CNN
-F 2 "MountingHole:MountingHole_2.7mm_M2.5_ISO14580_Pad" H 3050 800 50  0001 C CNN
+F 2 "SirBoardLibrary:MountingHole_M2.5_SirBoard" H 3050 800 50  0001 C CNN
 F 3 "~" H 3050 800 50  0001 C CNN
 	1    3050 800
@@
 F 0 "H2" H 3150 2045 50  0000 L CNN
 F 1 "MountingHole" H 3150 1955 50  0000 L CNN
-F 2 "MountingHole:MountingHole_2.7mm_M2.5_ISO14580_Pad" H 3050 2000 50  0001 C CNN
+F 2 "SirBoardLibrary:MountingHole_M2.5_SirBoard" H 3050 2000 50  0001 C CNN
 F 3 "~" H 3050 2000 50  0001 C CNN
 	1    3050 2000
@@
 F 0 "H3" H 2350 845 50  0000 L CNN
 F 1 "MountingHole" H 2350 755 50  0000 L CNN
-F 2 "MountingHole:MountingHole_2.7mm_M2.5_ISO14580_Pad" H 2250 800 50  0001 C CNN
+F 2 "SirBoardLibrary:MountingHole_M2.5_SirBoard" H 2250 800 50  0001 C CNN
 F 3 "~" H 2250 800 50  0001 C CNN
 	1    2250 800
@@
 F 0 "H4" H 2350 2045 50  0000 L CNN
 F 1 "MountingHole" H 2350 1955 50  0000 L CNN
-F 2 "MountingHole:MountingHole_2.7mm_M2.5_ISO14580_Pad" H 2250 2000 50  0001 C CNN
+F 2 "SirBoardLibrary:MountingHole_M2.5_SirBoard" H 2250 2000 50  0001 C CNN
 F 3 "~" H 2250 2000 50  0001 C CNN
 	1    2250 2000
