File: CR1220/CR1220.sch (KiCad schematic (older format))
At the start: 6 parts, among them J1 Conn_01x04

Commit message: Part Numbers Added
Parts:
- BT1: Part (none) -> C238097
Changed lines of the file:
@@
 F 2 "Battery:BatteryHolder_Keystone_3000_1x12mm" V 2150 1460 50  0001 C CNN
 F 3 "~" V 2150 1460 50  0001 C CNN
+F 4 "C238097" H 2150 1400 50  0001 C CNN "Part"
 	1    2150 1400
 	1    0    0    -1

Commit message: Board Redesign
Parts:
- H1, H2, H3, H4: footprint MountingHole:MountingHole_2.7mm_M2.5_ISO14580_Pad -> SirBoardLibrary:MountingHole_M2.5_SirBoard
Changed lines of the file:
@@
 F 0 "H1" H 3100 795 50  0000 L CNN
 F 1 "MountingHole" H 3100 705 50  0000 L CNN
-F 2 "MountingHole:MountingHole_2.7mm_M2.5_ISO14580_Pad" H 3000 750 50  0001 C CNN
+F 2 "SirBoardLibrary:MountingHole_M2.5_SirBoard" H 3000 750 50  0001 C CNN
 F 3 "~" H 3000 750 50  0001 C CNN
 	1    3000 750
@@
 F 0 "H2" H 3100 1995 50  0000 L CNN
 F 1 "MountingHole" H 3100 1905 50  0000 L CNN
-F 2 "MountingHole:MountingHole_2.7mm_M2.5_ISO14580_Pad" H 3000 1950 50  0001 C CNN
+F 2 "SirBoardLibrary:MountingHole_M2.5_SirBoard" H 3000 1950 50  0001 C CNN
 F 3 "~" H 3000 1950 50  0001 C CNN
 	1    3000 1950
@@
 F 0 "H3" H 2300 795 50  0000 L CNN
 F 1 "MountingHole" H 2300 705 50  0000 L CNN
-F 2 "MountingHole:MountingHole_2.7mm_M2.5_ISO14580_Pad" H 2200 750 50  0001 C CNN
+F 2 "SirBoardLibrary:MountingHole_M2.5_SirBoard" H 2200 750 50  0001 C CNN
 F 3 "~" H 2200 750 50  0001 C CNN
 	1    2200 750
@@
 F 0 "H4" H 2300 1995 50  0000 L CNN
 F 1 "MountingHole" H 2300 1905 50  0000 L CNN
-F 2 "MountingHole:MountingHole_2.7mm_M2.5_ISO14580_Pad" H 2200 1950 50  0001 C CNN
+F 2 "SirBoardLibrary:MountingHole_M2.5_SirBoard" H 2200 1950 50  0001 C CNN
 F 3 "~" H 2200 1950 50  0001 C CNN
 	1    2200 1950
