File: MicroSD_DualVoltage/MicroSD_DualVoltage.sch (KiCad schematic (older format))
At the start: 18 parts, among them J1 Conn_01x08, J3 Micro_SD_Card_Det, U1 AP7365, U2 TXB0104PW

Commit message: Part Numbers Added
Parts:
- C1, C2: Part (none) -> C29936
- C3, C4: Part (none) -> C42998
- D1: Part (none) -> C205443
- J3: Part (none) -> C114218
- R1: Part (none) -> C227816
- R2: value 12K5 -> 12K4; Part (none) -> C139128
- R3: Part (none) -> C99198
- R6: Part (none) -> C25585
- U1: Part (none) -> C264087
- U2: Part (none) -> C60708
Changed lines of the file:
@@
 F 2 "Connector_Card:microSD_HC_Hirose_DM3AT-SF-PEJM5" H 8500 4100 50  0001 C CNN
 F 3 "https://www.hirose.com/product/en/download_file/key_name/DM3/category/Catalog/doc_file_id/49662/?file_category_id=4&item_id=195&is_series=1" H 6450 3500 50  0001 C CNN
+F 4 "C114218" H 6450 3400 50  0001 C CNN "Part"
 	1    6450 3400
 	1    0    0    -1
@@
 F 2 "Package_TO_SOT_SMD:SOT-23-5" H 4900 6950 50  0001 C CNN
 F 3 "" H 4900 6950 50  0001 C CNN
+F 4 "C264087" H 4850 5950 50  0001 C CNN "Part"
 	1    4850 5950
 	1    0    0    -1
@@
 F 2 "Capacitor_SMD:C_0603_1608Metric" H 4288 5350 50  0001 C CNN
 F 3 "~" H 4250 5500 50  0001 C CNN
+F 4 "C29936" H 4250 5500 50  0001 C CNN "Part"
 	1    4250 5500
 	1    0    0    -1
@@
 F 2 "Capacitor_SMD:C_0603_1608Metric" H 5538 5350 50  0001 C CNN
 F 3 "~" H 5500 5500 50  0001 C CNN
+F 4 "C29936" H 5500 5500 50  0001 C CNN "Part"
 	1    5500 5500
 	1    0    0    -1
@@
 F 2 "Resistor_SMD:R_0603_1608Metric" V 3090 5140 50  0001 C CNN
 F 3 "~" H 3050 5150 50  0001 C CNN
+F 4 "C227816" H 3050 5150 50  0001 C CNN "Part"
 	1    3050 5150
 	1    0    0    -1
@@
 F 2 "Resistor_SMD:R_0603_1608Metric" V 3290 5790 50  0001 C CNN
 F 3 "~" H 3250 5800 50  0001 C CNN
+F 4 "C99198" H 3250 5800 50  0001 C CNN "Part"
 	1    3250 5800
 	1    0    0    -1
@@
 F 2 "Resistor_SMD:R_0603_1608Metric" V 4590 4540 50  0001 C CNN
 F 3 "~" H 4550 4550 50  0001 C CNN
+F 4 "C25585" V 4550 4550 50  0001 C CNN "Part"
 	1    4550 4550
 	0    -1   -1   0
@@
 F 2 "LED_SMD:LED_0603_1608Metric" H 4950 4550 50  0001 C CNN
 F 3 "~" H 4950 4550 50  0001 C CNN
+F 4 "C205443" H 4950 4550 50  0001 C CNN "Part"
 	1    4950 4550
 	-1   0    0    1
@@
 P 3450 5150
 F 0 "R2" H 3518 5195 50  0000 L CNN
-F 1 "12K5" H 3518 5105 50  0000 L CNN
+F 1 "12K4" H 3518 5105 50  0000 L CNN
 F 2 "Resistor_SMD:R_0603_1608Metric" V 3490 5140 50  0001 C CNN
 F 3 "~" H 3450 5150 50  0001 C CNN
+F 4 "C139128" H 3450 5150 50  0001 C CNN "Part"
 	1    3450 5150
 	1    0    0    -1
@@
 F 2 "Package_SO:TSSOP-14_4.4x5mm_P0.65mm" H 3700 2550 50  0001 C CNN
 F 3 "http://www.ti.com/lit/ds/symlink/txb0104.pdf" H 3810 3395 50  0001 C CNN
+F 4 "C60708" H 3700 3300 50  0001 C CNN "Part"
 	1    3700 3300
 	-1   0    0    -1
@@
 F 2 "Capacitor_SMD:C_0603_1608Metric" H 4538 2550 50  0001 C CNN
 F 3 "~" H 4500 2700 50  0001 C CNN
+F 4 "C42998" H 4500 2700 50  0001 C CNN "Part"
 	1    4500 2700
 	1    0    0    -1
@@
 F 2 "Capacitor_SMD:C_0603_1608Metric" H 2938 2550 50  0001 C CNN
 F 3 "~" H 2900 2700 50  0001 C CNN
+F 4 "C42998" H 2900 2700 50  0001 C CNN "Part"
 	1    2900 2700
 	1    0    0    -1

Commit message: Schematic PDF and 3D Renders added
Parts:
- U1: symbol U.FL-R-SMT(01):AP7365 -> MicroSD_DualVoltage-rescue:AP7365-U.FL-R-SMT(01)
Changed lines of the file:
@@
 $EndComp
 $Comp
-L U.FL-R-SMT(01):AP7365 U1
+L MicroSD_DualVoltage-rescue:AP7365-U.FL-R-SMT(01) U1
 U 1 1 5DB62551
 P 4850 5950

Commit message: Board Redesign
Parts:
- removed C1, C2: 1uF, Capacitor_SMD:C_0603_1608Metric, symbol Device:CP
- added C1, C2: 10uF, Capacitor_SMD:C_0805_2012Metric, symbol Device:C
- added R4: 10K, Resistor_SMD:R_0603_1608Metric, symbol Device:R_US
- H1, H2, H3, H4: footprint MountingHole:MountingHole_2.7mm_M2.5_ISO14580_Pad -> SirBoardLibrary:MountingHole_M2.5_SirBoard
Connections:
- net DETB is gone; now on net VOUT: J3.9 (DET_B)
- net DETA: now also R4.1
- net GND: now also C1.2, C2.2, R4.2
- net VIN: now also C1.1
- net VOUT: now also C2.1
Other:
- moved on the sheet: C3, C4, D1, H1, J1, J3, JP1, R1, R2, R3, R6, U1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
