File: MicroUSB/MicroUSB.sch (KiCad schematic (older format))
At the start: 4 parts, among them J1 USB_B_Micro, J2 Conn_01x05

Commit message: Part Numbers Added
Parts:
- J1: Part (none) -> C132560
Changed lines of the file:
@@
 F 2 "Connector_USB:USB_Micro-B_Molex_47346-0001" H 2450 1300 50  0001 C CNN
 F 3 "~" H 2450 1300 50  0001 C CNN
+F 4 "C132560" H 2300 1350 50  0001 C CNN "Part"
 	1    2300 1350
 	1    0    0    -1

Commit message: Board Redesign
Parts:
- H1, H2: footprint MountingHole:MountingHole_2.7mm_M2.5_ISO14580_Pad -> SirBoardLibrary:MountingHole_M2.5_SirBoard
Connections:
- net VBus: now reaches J1.1 (VBUS), J2.1 (Pin_1)
- net D-: now reaches J1.2 (D-), J2.2 (Pin_2)
- net D+: now reaches J1.3 (D+), J2.3 (Pin_3)
- net ID: now reaches J1.4 (ID), J2.4 (Pin_4)
- net GND: now reaches J1.5 (GND), J1.6 (Shield), J2.5 (Pin_5)
Changed lines of the file:
@@
 F 0 "H1" H 2350 795 50  0000 L CNN
 F 1 "MountingHole" H 2350 705 50  0000 L CNN
-F 2 "MountingHole:MountingHole_2.7mm_M2.5_ISO14580_Pad" H 2250 750 50  0001 C CNN
+F 2 "SirBoardLibrary:MountingHole_M2.5_SirBoard" H 2250 750 50  0001 C CNN
 F 3 "~" H 2250 750 50  0001 C CNN
 	1    2250 750
@@
 $Comp
 L Mechanical:MountingHole H2
-U 1 1 5DB39176
-P 2250 1950
-F 0 "H2" H 2350 1995 50  0000 L CNN
-F 1 "MountingHole" H 2350 1905 50  0000 L CNN
-F 2 "MountingHole:MountingHole_2.7mm_M2.5_ISO14580_Pad" H 2250 1950 50  0001 C CNN
-F 3 "~" H 2250 1950 50  0001 C CNN
-	1    2250 1950
+U 1 1 5E38278B
+P 2275 2050
+F 0 "H2" H 2375 2095 50  0000 L CNN
+F 1 "MountingHole" H 2375 2005 50  0000 L CNN
+F 2 "SirBoardLibrary:MountingHole_M2.5_SirBoard" H 2275 2050 50  0001 C CNN
+F 3 "~" H 2275 2050 50  0001 C CNN
+	1    2275 2050
 	1    0    0    -1
 $EndComp
+Text Label 2625 1150 0    50   ~ 0
+VBus
+Text Label 2625 1350 0    50   ~ 0
+D+
+Text Label 2625 1450 0    50   ~ 0
+D-
+Text Label 2625 1550 0    50   ~ 0
+ID
+Text Label 2625 1750 0    50   ~ 0
+GND
 $EndSCHEMATC
