File: MiniUSB/MiniUSB.sch (KiCad schematic (older format))
At the start: 4 parts, among them J1 USB_B_Micro, J2 Conn_01x05

Commit message: Part Numbers Added
Parts:
- J1: value USB_B_Micro -> USB_B_Mini; footprint Connector_USB:USB_Mini-B_Lumberg_2486_01_Horizontal -> SirBoardLibrary:SirBoard_USB_Mini-B; Part (none) -> C69074
Changed lines of the file:
@@
 P 2450 1350
 F 0 "J1" H 2506 1815 50  0000 C CNN
-F 1 "USB_B_Micro" H 2506 1725 50  0000 C CNN
-F 2 "Connector_USB:USB_Mini-B_Lumberg_2486_01_Horizontal" H 2600 1300 50  0001 C CNN
+F 1 "USB_B_Mini" H 2506 1725 50  0000 C CNN
+F 2 "SirBoardLibrary:SirBoard_USB_Mini-B" H 2600 1300 50  0001 C CNN
 F 3 "~" H 2600 1300 50  0001 C CNN
+F 4 "C69074" H 2450 1350 50  0001 C CNN "Part"
 	1    2450 1350
 	1    0    0    -1

Commit message: Board Redesign
Parts:
- H1, H2: footprint MountingHole:MountingHole_2.7mm_M2.5_ISO14580_Pad -> SirBoardLibrary:MountingHole_M2.5_SirBoard
Connections:
- net VBus: now reaches J1.1 (VBUS), J2.1 (Pin_1)
- net D-: now reaches J1.2 (D-), J2.2 (Pin_2)
- net D+: now reaches J1.3 (D+), J2.3 (Pin_3)
- net ID: now reaches J1.4 (ID), J2.4 (Pin_4)
- net GND: now reaches J1.5 (GND), J1.6 (Shield), J2.5 (Pin_5)
Changed lines of the file:
@@
 Connection ~ 2450 1750
-$Comp
-L Mechanical:MountingHole H1
-U 1 1 5DB38589
-P 2400 750
-F 0 "H1" H 2500 795 50  0000 L CNN
-F 1 "MountingHole" H 2500 705 50  0000 L CNN
-F 2 "MountingHole:MountingHole_2.7mm_M2.5_ISO14580_Pad" H 2400 750 50  0001 C CNN
-F 3 "~" H 2400 750 50  0001 C CNN
-	1    2400 750
-	1    0    0    -1
-$EndComp
 $Comp
 L Mechanical:MountingHole H2
@@
 F 0 "H2" H 2500 1995 50  0000 L CNN
 F 1 "MountingHole" H 2500 1905 50  0000 L CNN
-F 2 "MountingHole:MountingHole_2.7mm_M2.5_ISO14580_Pad" H 2400 1950 50  0001 C CNN
+F 2 "SirBoardLibrary:MountingHole_M2.5_SirBoard" H 2400 1950 50  0001 C CNN
 F 3 "~" H 2400 1950 50  0001 C CNN
 	1    2400 1950
 	1    0    0    -1
 $EndComp
+Text Label 2800 1150 0    50   ~ 0
+VBus
+Text Label 2825 1350 0    50   ~ 0
+D+
+Text Label 2825 1450 0    50   ~ 0
+D-
+Text Label 2825 1550 0    50   ~ 0
+ID
+Text Label 2825 1750 0    50   ~ 0
+GND
+$Comp
+L Mechanical:MountingHole H1
+U 1 1 5E383516
+P 2400 775
+F 0 "H1" H 2500 820 50  0000 L CNN
+F 1 "MountingHole" H 2500 730 50  0000 L CNN
+F 2 "SirBoardLibrary:MountingHole_M2.5_SirBoard" H 2400 775 50  0001 C CNN
+F 3 "~" H 2400 775 50  0001 C CNN
+	1    2400 775
+	1    0    0    -1
+$EndComp
