File: SOT6/SOT6.kicad_pcb (KiCad board)
At the start: 2 copper layers, 8.9 x 11.4 mm, 5 parts, among them J1 Conn_01x03, J2 Conn_01x03, J3 Conn_02x03_Counter_Clockwise, J4 Conn_02x03_Counter_Clockwise

Commit message: Schematic PDF and 3D Renders added
Parts:
- J4: footprint Package_TO_SOT_SMD:SOT-363_SC-70-6 -> Package_TO_SOT_SMD:SOT-363_SC-70-6_Handsoldering
Changed lines of the file:
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@@
     (34 B.Paste user hide)
     (35 F.Paste user hide)
-    (36 B.SilkS user)
-    (37 F.SilkS user)
+    (36 B.SilkS user hide)
+    (37 F.SilkS user hide)
     (38 B.Mask user hide)
     (39 F.Mask user hide)
@@
     (add_net "Net-(J2-Pad2)")
     (add_net "Net-(J2-Pad3)")
+  )
+  (module Package_TO_SOT_SMD:SOT-363_SC-70-6_Handsoldering (layer B.Cu)
+    (at 68.072 36.83 270)
+    (descr "SOT-363, SC-70-6, Handsoldering")
+    (tags "SOT-363 SC-70-6 Handsoldering")
+    (attr smd)
+    (fp_text reference J4 (at 0 2 90) (layer B.SilkS) hide
+      (effects (font (size 1 1) (thickness 0.15)) (justify mirror))
+    )
+    (fp_text value Conn_02x03_Counter_Clockwise (at 0 -2 270) (layer B.Fab)
+      (effects (font (size 1 1) (thickness 0.15)) (justify mirror))
+    )
+    (fp_line (start -0.175 1.1) (end -0.675 0.6) (layer B.Fab) (width 0.1))
+    (fp_line (start 0.675 -1.1) (end -0.675 -1.1) (layer B.Fab) (width 0.1))
+    (fp_line (start 0.675 1.1) (end 0.675 -1.1) (layer B.Fab) (width 0.1))
+    (fp_line (start -0.675 0.6) (end -0.675 -1.1) (layer B.Fab) (width 0.1))
+    (fp_line (start 0.675 1.1) (end -0.175 1.1) (layer B.Fab) (width 0.1))
+    (fp_line (start -2.4 1.4) (end 2.4 1.4) (layer B.CrtYd) (width 0.05))
+    (fp_line (start -2.4 1.4) (end -2.4 -1.4) (layer B.CrtYd) (width 0.05))
+    (fp_line (start 2.4 -1.4) (end 2.4 1.4) (layer B.CrtYd) (width 0.05))
+    (fp_line (start -0.7 -1.16) (end 0.7 -1.16) (layer B.SilkS) (width 0.12))
+    (fp_line (start 0.7 1.16) (end -1.2 1.16) (layer B.SilkS) (width 0.12))
+    (fp_line (start -2.4 -1.4) (end 2.4 -1.4) (layer B.CrtYd) (width 0.05))
+    (fp_text user %R (at 0 0 180) (layer B.Fab)
+      (effects (font (size 0.5 0.5) (thickness 0.075)) (justify mirror))
+    )
+    (pad 6 smd rect (at 1.33 0.65 270) (size 1.5 0.4) (layers B.Cu B.Paste B.Mask)
+      (net 6 "Net-(J2-Pad1)"))
+    (pad 5 smd rect (at 1.33 0 270) (size 1.5 0.4) (layers B.Cu B.Paste B.Mask)
+      (net 5 "Net-(J2-Pad2)"))
+    (pad 4 smd rect (at 1.33 -0.65 270) (size 1.5 0.4) (layers B.Cu B.Paste B.Mask)
+      (net 4 "Net-(J2-Pad3)"))
+    (pad 3 smd rect (at -1.33 -0.65 270) (size 1.5 0.4) (layers B.Cu B.Paste B.Mask)
+      (net 1 "Net-(J1-Pad3)"))
+    (pad 2 smd rect (at -1.33 0 270) (size 1.5 0.4) (layers B.Cu B.Paste B.Mask)
+      (net 2 "Net-(J1-Pad2)"))
+    (pad 1 smd rect (at -1.33 0.65 270) (size 1.5 0.4) (layers B.Cu B.Paste B.Mask)
+      (net 3 "Net-(J1-Pad1)"))
+    (model ${KISYS3DMOD}/Package_TO_SOT_SMD.3dshapes/SOT-363_SC-70-6.wrl
+      (at (xyz 0 0 0))
+      (scale (xyz 1 1 1))
+      (rotate (xyz 0 0 0))
+    )
   )
   (module Package_TO_SOT_SMD:SOT-23-6_Handsoldering (layer F.Cu)
@@
       (xy 0.01011 1.901832) (xy 0.176764 1.897837)) (layer B.SilkS) (width 0.01))
   )
-  (module Package_TO_SOT_SMD:SOT-363_SC-70-6 (layer B.Cu)
-    (at 68.072 36.83 270)
-    (descr "SOT-363, SC-70-6")
-    (tags "SOT-363 SC-70-6")
-    (attr smd)
-    (fp_text reference J4 (at 0 2 90) (layer B.SilkS) hide
-      (effects (font (size 1 1) (thickness 0.15)) (justify mirror))
-    )
-    (fp_text value Conn_02x03_Counter_Clockwise (at 0 -2 270) (layer B.Fab)
-      (effects (font (size 1 1) (thickness 0.15)) (justify mirror))
-    )
-    (fp_line (start -0.175 1.1) (end -0.675 0.6) (layer B.Fab) (width 0.1))
-    (fp_line (start 0.675 -1.1) (end -0.675 -1.1) (layer B.Fab) (width 0.1))
-    (fp_line (start 0.675 1.1) (end 0.675 -1.1) (layer B.Fab) (width 0.1))
-    (fp_line (start -1.6 -1.4) (end 1.6 -1.4) (layer B.CrtYd) (width 0.05))
-    (fp_line (start -0.675 0.6) (end -0.675 -1.1) (layer B.Fab) (width 0.1))
-    (fp_line (start 0.675 1.1) (end -0.175 1.1) (layer B.Fab) (width 0.1))
-    (fp_line (start -1.6 1.4) (end 1.6 1.4) (layer B.CrtYd) (width 0.05))
-    (fp_line (start -1.6 1.4) (end -1.6 -1.4) (layer B.CrtYd) (width 0.05))
-    (fp_line (start 1.6 -1.4) (end 1.6 1.4) (layer B.CrtYd) (width 0.05))
-    (fp_line (start -0.7 -1.16) (end 0.7 -1.16) (layer B.SilkS) (width 0.12))
-    (fp_line (start 0.7 1.16) (end -1.2 1.16) (layer B.SilkS) (width 0.12))
-    (fp_text user %R (at 0 0 180) (layer B.Fab)
-      (effects (font (size 0.5 0.5) (thickness 0.075)) (justify mirror))
-    )
-    (pad 6 smd rect (at 0.95 0.65 270) (size 0.65 0.4) (layers B.Cu B.Paste B.Mask)
-      (net 6 "Net-(J2-Pad1)"))
-    (pad 4 smd rect (at 0.95 -0.65 270) (size 0.65 0.4) (layers B.Cu B.Paste B.Mask)
-      (net 4 "Net-(J2-Pad3)"))
-    (pad 2 smd rect (at -0.95 0 270) (size 0.65 0.4) (layers B.Cu B.Paste B.Mask)
-      (net 2 "Net-(J1-Pad2)"))
-    (pad 5 smd rect (at 0.95 0 270) (size 0.65 0.4) (layers B.Cu B.Paste B.Mask)
-      (net 5 "Net-(J2-Pad2)"))
-    (pad 3 smd rect (at -0.95 -0.65 270) (size 0.65 0.4) (layers B.Cu B.Paste B.Mask)
-      (net 1 "Net-(J1-Pad3)"))
-    (pad 1 smd rect (at -0.95 0.65 270) (size 0.65 0.4) (layers B.Cu B.Paste B.Mask)
-      (net 3 "Net-(J1-Pad1)"))
-    (model ${KISYS3DMOD}/Package_TO_SOT_SMD.3dshapes/SOT-363_SC-70-6.wrl
-      (at (xyz 0 0 0))
-      (scale (xyz 1 1 1))
-      (rotate (xyz 0 0 0))
-    )
-  )
   (module Connector_PinHeader_2.54mm:PinHeader_1x03_P2.54mm_Vertical (layer F.Cu)

Commit message: Board Updates
Parts:
- moved J3 2.54 mm to (65.5, 36.8)
- moved J4 2.54 mm to (65.5, 36.8)
- moved J1 2.54 mm to (63.0, 33.0)
- moved J2 2.54 mm to (63.0, 40.6)
- moved G*** 2.29 mm to (63.0, 36.8)
Other:
- board size 8.9 x 11.4 mm -> 7.6 x 10.2 mm
