File: USB_C/USBC.sch (KiCad schematic (older format))
At the start: 6 parts, among them J1 USB_C_Receptacle_USB2.0, J2 Conn_01x08

Commit message: Part Numbers Added
Parts:
- J1: Part (none) -> C165948
- R1, R2: Part (none) -> C332117
Changed lines of the file:
@@
 F 2 "U_FL:USB_C" H 2500 1600 50  0001 C CNN
 F 3 "https://www.usb.org/sites/default/files/documents/usb_type-c.zip" H 2500 1600 50  0001 C CNN
+F 4 "C165948" H 2350 1600 50  0001 C CNN "Part"
 	1    2350 1600
 	1    0    0    -1
@@
 F 2 "Resistor_SMD:R_0805_2012Metric" V 3340 1190 50  0001 C CNN
 F 3 "~" H 3300 1200 50  0001 C CNN
+F 4 "C332117" V 3300 1200 50  0001 C CNN "Part"
 	1    3300 1200
 	0    1    1    0
@@
 F 2 "Resistor_SMD:R_0805_2012Metric" V 3340 1290 50  0001 C CNN
 F 3 "~" H 3300 1300 50  0001 C CNN
+F 4 "C332117" V 3300 1300 50  0001 C CNN "Part"
 	1    3300 1300
 	0    1    1    0

Commit message: Board Redesign
Parts:
- H1, H2: footprint MountingHole:MountingHole_2.7mm_M2.5_ISO14580_Pad -> SirBoardLibrary:MountingHole_M2.5_SirBoard
- J1: footprint U_FL:USB_C -> SirBoardLibrary:USB_C
Connections:
- net D+: now also J2.5 (Pin_5); no longer J2.6 (Pin_6)
- net D-: now also J2.6 (Pin_6); no longer J2.5 (Pin_5)
- net SBU1: now also J2.4 (Pin_4); no longer J2.8 (Pin_8)
- net SBU2: now also J2.8 (Pin_8); no longer J2.4 (Pin_4)
Other:
- moved on the sheet: H1
Changed lines of the file:
@@
 L Mechanical:MountingHole H1
 U 1 1 5DB38589
-P 1750 1000
-F 0 "H1" H 1850 1045 50  0000 L CNN
-F 1 "MountingHole" H 1850 955 50  0000 L CNN
-F 2 "MountingHole:MountingHole_2.7mm_M2.5_ISO14580_Pad" H 1750 1000 50  0001 C CNN
-F 3 "~" H 1750 1000 50  0001 C CNN
-	1    1750 1000
-	-1   0    0    -1
-$EndComp
-$Comp
-L Mechanical:MountingHole H2
-U 1 1 5DB39176
-P 1750 2200
-F 0 "H2" H 1850 2245 50  0000 L CNN
-F 1 "MountingHole" H 1850 2155 50  0000 L CNN
-F 2 "MountingHole:MountingHole_2.7mm_M2.5_ISO14580_Pad" H 1750 2200 50  0001 C CNN
-F 3 "~" H 1750 2200 50  0001 C CNN
-	1    1750 2200
+P 1725 1425
+F 0 "H1" H 1825 1470 50  0000 L CNN
+F 1 "MountingHole" H 1825 1380 50  0000 L CNN
+F 2 "SirBoardLibrary:MountingHole_M2.5_SirBoard" H 1725 1425 50  0001 C CNN
+F 3 "~" H 1725 1425 50  0001 C CNN
+	1    1725 1425
 	-1   0    0    -1
 $EndComp
@@
 F 0 "J1" H 2456 2465 50  0000 C CNN
 F 1 "USB_C_Receptacle_USB2.0" H 2456 2375 50  0000 C CNN
-F 2 "U_FL:USB_C" H 2500 1600 50  0001 C CNN
+F 2 "SirBoardLibrary:USB_C" H 2500 1600 50  0001 C CNN
 F 3 "https://www.usb.org/sites/default/files/documents/usb_type-c.zip" H 2500 1600 50  0001 C CNN
 F 4 "C165948" H 2350 1600 50  0001 C CNN "Part"
@@
 	3100 1300 3150 1300
 Wire Wire Line
-	2950 2200 3650 2200
-Wire Wire Line
-	3650 2200 3650 1500
-Wire Wire Line
 	3650 1500 4050 1500
 Wire Wire Line
 	3400 1500 3400 1600
-Wire Wire Line
-	3400 1600 4050 1600
 Wire Wire Line
 	2950 1800 3000 1800
@@
 	3050 1200 3150 1200
 Wire Wire Line
-	2950 2100 4050 2100
-Wire Wire Line
-	4050 2100 4050 1900
-Wire Wire Line
 	2950 1700 3000 1700
 Wire Wire Line
@@
 Wire Wire Line
 	3000 1800 3000 1700
-Connection ~ 3000 1700
-Wire Wire Line
-	3000 1700 4050 1700
 Wire Wire Line
 	2950 1600 3000 1600
@@
 Text Label 3700 1400 0    50   ~ 0
 CC2
-Text Label 3700 1500 0    50   ~ 0
+Text Label 3700 2200 0    50   ~ 0
 SBU2
 Text Label 3700 1600 0    50   ~ 0
-D-
-Text Label 3700 1700 0    50   ~ 0
 D+
 Text Label 3700 1800 0    50   ~ 0
 CC1
-Text Label 3700 2100 0    50   ~ 0
+Text Label 3700 1500 0    50   ~ 0
 SBU1
+$Comp
+L Mechanical:MountingHole H2
+U 1 1 5E3F3E24
+P 1725 1750
+F 0 "H2" H 1825 1795 50  0000 L CNN
+F 1 "MountingHole" H 1825 1705 50  0000 L CNN
+F 2 "SirBoardLibrary:MountingHole_M2.5_SirBoard" H 1725 1750 50  0001 C CNN
+F 3 "~" H 1725 1750 50  0001 C CNN
+	1    1725 1750
+	-1   0    0    -1
+$EndComp
+Wire Wire Line
+	3000 1700 3400 1700
+Wire Wire Line
+	3400 1700 3450 1650
+Wire Wire Line
+	3500 1600 4050 1600
+Connection ~ 3000 1700
+Wire Wire Line
+	3450 1650 3500 1600
+Wire Wire Line
+	3400 1600 3500 1700
+Wire Wire Line
+	3500 1700 4050 1700
+Text Label 3700 1700 0    50   ~ 0
+D-
+Wire Wire Line
+	4050 1900 4050 2200
+Wire Wire Line
+	2950 2200 4050 2200
+Wire Wire Line
+	2950 2100 3650 2100
+Wire Wire Line
+	3650 2100 3650 1500
 $EndSCHEMATC

Commit message: Breakout Boards Revision 2
Renders updated, silkscreen text improved, blurry silkscreen items removed/resized.
Parts:
- R1, R2: footprint Resistor_SMD:R_0805_2012Metric -> Resistor_SMD:R_0603_1608Metric
Changed lines of the file:
@@
 F 0 "R1" V 3097 1200 50  0000 C CNN
 F 1 "5K1" V 3187 1200 50  0000 C CNN
-F 2 "Resistor_SMD:R_0805_2012Metric" V 3340 1190 50  0001 C CNN
+F 2 "Resistor_SMD:R_0603_1608Metric" V 3340 1190 50  0001 C CNN
 F 3 "~" H 3300 1200 50  0001 C CNN
 F 4 "C332117" V 3300 1200 50  0001 C CNN "Part"
@@
 F 0 "R2" V 3503 1300 50  0000 C CNN
 F 1 "5K1" V 3413 1300 50  0000 C CNN
-F 2 "Resistor_SMD:R_0805_2012Metric" V 3340 1290 50  0001 C CNN
+F 2 "Resistor_SMD:R_0603_1608Metric" V 3340 1290 50  0001 C CNN
 F 3 "~" H 3300 1300 50  0001 C CNN
 F 4 "C332117" V 3300 1300 50  0001 C CNN "Part"
